File: pcb/bypass_mod.kicad_pcb (KiCad board)
At the start: 2 copper layers, 16 x 19.8 mm, 10 parts, among them J1 isp, J2 switch_conn, J3 io_conn, Q1 2N7002, U1 L78L05_SOT89, U2 ATtiny85-20S

Commit message: Updates
Parts:
- U2: footprint Package_SO:SOIC-8W_5.3x5.3mm_P1.27mm -> kicad library:SOICxDIP
- moved JP1 5.22 mm to (143.1, 109.2), turned to 180 degrees
- moved J2 4.25 mm to (152.2, 109.2)
- moved U2 1.94 mm to (149.2, 102.0)
- moved J1 1.52 mm to (141.7, 102.0), turned to 90 degrees
- moved G*** 0.07 mm to (147.2, 93.0)
Routing:
- net /mosi: track 3.88 -> 19.5 mm
- net /sck: track 27.5 -> 18.3 mm, vias 2 -> 0
- net /bypass: track 4.46 -> 10.4 mm
- net +5V: track 14.7 -> 20.5 mm
- net Net-(JP1-A): track 9.51 -> 14.4 mm, vias 1 -> 0
- net /miso: track 9.82 -> 13.4 mm, vias 2 -> 0
- net GND: track 25.0 -> 23.1 mm, vias 1 -> 0
- net /rst: track 22.7 -> 21.6 mm
Other:
- board size 16 x 19.8 mm -> 16 x 23.8 mm
- board text added: "rev2"
- board text added: "switching mod"
- board text removed: "switching mod rev1"
