File: pcb/bypass_mod.kicad_sch (KiCad schematic)
At the start: 9 parts, among them J1 isp, J2 switch_conn, J3 io_conn, Q1 2N7002, U1 L78L05_SOT89, U2 ATtiny85-20S

Commit message: Updates
Parts:
- U2: footprint Package_SO:SOIC-8W_5.3x5.3mm_P1.27mm -> kicad library:SOICxDIP
Changed lines of the file:
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@@
       (effects (font (size 1.27 1.27)) (justify right))
     )
-    (property "Footprint" "Package_SO:SOIC-8W_5.3x5.3mm_P1.27mm" (at 93.98 76.2 0)
+    (property "Footprint" "kicad library:SOICxDIP" (at 93.98 76.2 0)
       (effects (font (size 1.27 1.27) italic) hide)
     )
